File: KiCAD/YeroKB.kicad_sch (KiCad schematic)
At the start: 190 parts, among them SW1 SW_Push, U1 nRF52840

Commit message: Added all column names
Parts:
- added D91, D92, D93, D94, D95, D96: D_Small, symbol Device:D_Small
- added MX91, MX92, MX93, MX94, MX95, MX96: MX-NoLED, symbol MX_Alps_Hybrid:MX-NoLED
Connections:
- net COL0: no longer MX10.1 (COL), MX11.1 (COL), MX12.1 (COL), MX13.1 (COL), MX14.1 (COL), MX15.1 (COL), MX16.1 (COL), MX17.1 (COL), MX18.1 (COL), MX19.1 (COL), MX20.1 (COL), MX21.1 (COL), MX22.1 (COL), MX23.1 (COL), MX24.1 (COL), MX25.1 (COL), MX26.1 (COL), MX27.1 (COL), MX28.1 (COL), MX29.1 (COL), MX30.1 (COL), MX31.1 (COL), MX32.1 (COL), MX33.1 (COL), MX34.1 (COL), MX35.1 (COL), MX36.1 (COL), MX37.1 (COL), MX38.1 (COL), MX39.1 (COL), MX40.1 (COL), MX41.1 (COL), MX42.1 (COL), MX43.1 (COL), MX44.1 (COL), MX45.1 (COL), MX46.1 (COL), MX47.1 (COL), MX48.1 (COL), MX49.1 (COL), MX50.1 (COL), MX51.1 (COL), MX52.1 (COL), MX53.1 (COL), MX54.1 (COL), MX55.1 (COL), MX56.1 (COL), MX57.1 (COL), MX58.1 (COL), MX59.1 (COL), MX60.1 (COL), MX61.1 (COL), MX62.1 (COL), MX63.1 (COL), MX64.1 (COL), MX65.1 (COL), MX66.1 (COL), MX67.1 (COL), MX68.1 (COL), MX69.1 (COL), MX7.1 (COL), MX70.1 (COL), MX71.1 (COL), MX72.1 (COL), MX73.1 (COL), MX74.1 (COL), MX75.1 (COL), MX76.1 (COL), MX77.1 (COL), MX78.1 (COL), MX79.1 (COL), MX8.1 (COL), MX80.1 (COL), MX81.1 (COL), MX82.1 (COL), MX83.1 (COL), MX84.1 (COL), MX85.1 (COL), MX86.1 (COL), MX87.1 (COL), MX88.1 (COL), MX89.1 (COL), MX9.1 (COL), MX90.1 (COL)
- net ROW0: now also D91.1 (K)
- net ROW1: now also D92.1 (K)
- net ROW2: now also D93.1 (K)
- net ROW3: now also D94.1 (K)
- net ROW4: now also D95.1 (K)
- net ROW5: now also D96.1 (K)
- new net: D91.2 (A), MX91.2 (ROW)
- new net: D92.2 (A), MX92.2 (ROW)
- new net: D93.2 (A), MX93.2 (ROW)
- new net: D96.2 (A), MX96.2 (ROW)
- new net: D95.2 (A), MX95.2 (ROW)
- new net: D94.2 (A), MX94.2 (ROW)
- new net COL1: MX10.1 (COL), MX11.1 (COL), MX12.1 (COL), MX7.1 (COL), MX8.1 (COL), MX9.1 (COL)
- new net COL10: MX61.1 (COL), MX62.1 (COL), MX63.1 (COL), MX64.1 (COL), MX65.1 (COL), MX66.1 (COL)
- new net COL11: MX67.1 (COL), MX68.1 (COL), MX69.1 (COL), MX70.1 (COL), MX71.1 (COL), MX72.1 (COL)
- new net COL12: MX73.1 (COL), MX74.1 (COL), MX75.1 (COL), MX76.1 (COL), MX77.1 (COL), MX78.1 (COL)
- new net COL13: MX79.1 (COL), MX80.1 (COL), MX81.1 (COL), MX82.1 (COL), MX83.1 (COL), MX84.1 (COL)
- new net COL14: MX85.1 (COL), MX86.1 (COL), MX87.1 (COL), MX88.1 (COL), MX89.1 (COL), MX90.1 (COL)
- new net COL15: MX91.1 (COL), MX92.1 (COL), MX93.1 (COL), MX94.1 (COL), MX95.1 (COL), MX96.1 (COL)
- new net COL2: MX13.1 (COL), MX14.1 (COL), MX15.1 (COL), MX16.1 (COL), MX17.1 (COL), MX18.1 (COL)
- new net COL3: MX19.1 (COL), MX20.1 (COL), MX21.1 (COL), MX22.1 (COL), MX23.1 (COL), MX24.1 (COL)
- new net COL4: MX25.1 (COL), MX26.1 (COL), MX27.1 (COL), MX28.1 (COL), MX29.1 (COL), MX30.1 (COL)
- new net COL5: MX31.1 (COL), MX32.1 (COL), MX33.1 (COL), MX34.1 (COL), MX35.1 (COL), MX36.1 (COL)
- new net COL6: MX37.1 (COL), MX38.1 (COL), MX39.1 (COL), MX40.1 (COL), MX41.1 (COL), MX42.1 (COL)
- new net COL7: MX43.1 (COL), MX44.1 (COL), MX45.1 (COL), MX46.1 (COL), MX47.1 (COL), MX48.1 (COL)
- new net COL8: MX49.1 (COL), MX50.1 (COL), MX51.1 (COL), MX52.1 (COL), MX53.1 (COL), MX54.1 (COL)
- new net COL9: MX55.1 (COL), MX56.1 (COL), MX57.1 (COL), MX58.1 (COL), MX59.1 (COL), MX60.1 (COL)
Other:
- title: (none) -> YeroKB
